File: PCB/totem_0-3/totem_0_3.kicad_sch (KiCad schematic)
At the start: 88 parts, among them J1 MJ-4PP-9, J2 MJ-4PP-9, U1 xiao-ble, U2 xiao-ble

Commit message: Initial update from original
Parts:
- added DL17, DR20: D_Small, TOTEMlib:Diode_SOD123, symbol Device:D_Small
- added SWL17, SWR20: SW_Push_45deg, TOTEMlib:Kailh_socket_PG1350_optional, symbol Switch:SW_Push_45deg
- renumbered DL17 to DL18, DL18 to DL19, DL19 to DL20, SWL17 to SWL18, SWL18 to SWL19, SWL19 to SWL20
Connections:
- net COL1_L: now also SWL17.1
- net COL1_R: now also SWR17.1
- net COL2_R: now also SWR18.1; no longer SWR17.1
- net COL3_R: now also SWR19.1; no longer SWR18.1
- net COL4_R: now also SWR20.1; no longer SWR19.1
- net ROW3_L: now also DL17.1 (K)
- net ROW3_R: now also DR20.1 (K)
- new net: DL17.2 (A), SWL17.2
- new net: DR20.2 (A), SWR20.2
Other:
- moved on the sheet: DR17, DR18, DR19, SWR17, SWR18, SWR19
